Commit message: - atlas sinusoidal joint input

File: res/benchmark/Atlas-contact-benchmark/mujoco/robot1.urdf (robot description, URDF)
Before this commit: robot drc_skeleton, 46 links, 44 joints
Links:
- link l_foot_0: geometry collision box size=0.1 0.08 0.02; collision box size=0.227 0.133887 0.05
- link r_foot_0: geometry collision box size=0.1 0.08 0.02; collision box size=0.227 0.133887 0.05

File: res/benchmark/Atlas-contact-benchmark/ode-rai-dart/robot.urdf (robot description, URDF)
Before this commit: robot drc_skeleton, 44 links, 43 joints
Links:
- link l_foot: geometry collision box size=0.1 0.08 0.02; collision box size=0.227 0.133887 0.05
- link r_foot: geometry collision box size=0.1 0.08 0.02; collision box size=0.227 0.133887 0.05
